File: PCB/388_Project.sch (EAGLE design)
At the start: 37 parts, among them IC1 7824DT, U1 ATMEGA328P_TQFP

Commit message: Add files via upload
Parts:
- removed CN1: (no value), adafruit:DCBARRELSMT
- removed HEATER, LIGHT: RELAYPTH4, SparkFun-Electromechanical:RELAYPTH4
- removed Q4: (no value), adafruit:MOSFET-NREFLOW
- removed R8, R9: 150, resistor:R-US_M0805
- added CRYST: (no value), crystal:CRYSTALHC49UP
- added K1, K2: G5LE, ECE388:G5LE
- added R1, R2: 150, resistor:R-US_M0805
- added U$1: 2.1MMJACKTHM, ECE388:2.1MMJACKTHM
- Q1: device crystal:CRYSTALHC49U-V -> semicon-smd-ipc:NPN-TRANSISTOR_SOT23
- Q3: device semicon-smd-ipc:NPN-TRANSISTOR_SOT23 -> adafruit:MOSFET-NREFLOW
- R4: value 150 -> 120
- R6: value 10k -> 150
- R7: value 120 -> 10k
- X1: value (none) -> NC
- renumbered R10 to R3
Connections:
- net +12V: now also U$1.TIP; no longer CN1.PWR
- net +5V: now also K11.1, K21.1, R4.2; no longer HEATER.COIL1, LIGHT.COIL1, R7.2
- net FAN: now also R7.2; no longer R6.2
- net FAN_GND: now also Q3.D; no longer Q4.D
- net GND: now also Q1.C, Q3.S, R5.2, R6.2, U$1.RING, U$1.RING_SW; no longer CN1.GND, CN1.GNDBREAK, Q3.C, Q4.S, R8.2, R9.2
- net N$1: now also K12.O, TERMINAL-3.KL; no longer HEATER.NO, X1-1.KL
- net N$10: now also Q2.B, R2.2; no longer Q3.B, R5.2
- net N$11: now also K11.2, Q1.E; no longer LIGHT.COIL2, Q2.E
- net N$12: now also K21.2, Q2.E; no longer HEATER.COIL2, Q3.E
- net N$14: now also R5.1; no longer R8.1
- net N$15: now also R6.1; no longer R9.1
- net N$16: now also K22.O, X1-3.KL; no longer LIGHT.NO, TERMINAL-1.KL
- net N$17: now also K22.S, X1-1.KL; no longer LIGHT.MAIN, TERMINAL-2.KL
- net N$18: now also K22.P, X1-2.KL; no longer LIGHT.NC, TERMINAL-3.KL
- net N$2: now also Q3.G, R7.1; no longer Q4.G, R6.1
- net N$25: now also R4.1; no longer R7.1
- net N$3: now also CRYST.2; no longer Q1.2
- net N$4: now also CRYST.1; no longer Q1.1
- net N$5: now also K12.S, TERMINAL-1.KL; no longer HEATER.MAIN, X1-2.KL
- net N$6: now also K12.P, TERMINAL-2.KL; no longer HEATER.NC, X1-3.KL
- net N$7: now also R1.1; no longer R4.1
- net N$8: now also R2.1; no longer R5.1
- net N$9: now also Q1.B, R1.2; no longer Q2.B, R4.2
Other:
- moved on the sheet: Q2, R4, R5, R6, R7, TERMINAL-1, TERMINAL-2, TERMINAL-3, X1-1, X1-2, X1-3
